Commit message: update references to ur10_description

File: ur10_description/ur10.urdf (robot description, URDF)
Before this commit: robot ur10, 9 links, 8 joints
Links:
- link base_link: geometry collision mesh filename=package://ur10_description/meshes/ur10/collision/Base.dae; visual mesh filename=package://ur10_description/meshes/ur10/visual/Base.dae
- link forearm_link: geometry collision mesh filename=package://ur10_description/meshes/ur10/collision/Forearm.dae; visual mesh filename=package://ur10_description/meshes/ur10/visual/Forearm.dae
- link shoulder_link: geometry collision mesh filename=package://ur10_description/meshes/ur10/collision/Shoulder.d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; visual mesh filename=package://ur10_description/meshes/ur10/visual/Shoulder.dae
- link upper_arm_link: geometry collision mesh filename=package://ur10_description/meshes/ur10/collision/UpperArm.d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; visual mesh filename=package://ur10_description/meshes/ur10/visual/UpperArm.dae
- link wrist_1_link: geometry collision mesh filename=package://ur10_description/meshes/ur10/collision/Wrist1.dae; visual mesh filename=package://ur10_description/meshes/ur10/visual/Wrist1.dae
- link wrist_2_link: geometry collision mesh filename=package://ur10_description/meshes/ur10/collision/Wrist2.dae; visual mesh filename=package://ur10_description/meshes/ur10/visual/Wrist2.dae
- link wrist_3_link: geometry collision mesh filename=package://ur10_description/meshes/ur10/collision/Wrist3.dae; visual mesh filename=package://ur10_description/meshes/ur10/visual/Wrist3.dae
